File: base_pcb.kicad_pcb (KiCad board)
At the start: 2 copper layers, 3 parts, among them J1 Conn_01x20_Pin, J2 Conn_01x20_Pin

Commit message: Add STM pinouts
Parts:
- removed MotorController1: STM32F411_BP, ROBO:STM32F411-BP
- added B2: ~, MyCustoms:BNO085, F.Cu at (39.4, 29.2)
- added C1: 2.2u, Capacitor_SMD:C_0603_1608Metric_Pad1.08x0.95mm_HandSolder, F.Cu at (174.8, 103.1)
- added C10: 10u, Capacitor_SMD:C_0603_1608Metric_Pad1.08x0.95mm_HandSolder, F.Cu at (43.4, 140.5)
- added C11: 0.1u, Capacitor_SMD:C_0603_1608Metric_Pad1.08x0.95mm_HandSolder, F.Cu at (164.7, 46.2)
- added C13: 0.1u, Capacitor_SMD:C_0603_1608Metric_Pad1.08x0.95mm_HandSolder, F.Cu at (157.8, 46.7)
- added C2: 10u, Capacitor_SMD:C_0603_1608Metric_Pad1.08x0.95mm_HandSolder, F.Cu at (167.0, 110.7)
- added C5: 0.1u, Capacitor_SMD:C_0603_1608Metric_Pad1.08x0.95mm_HandSolder, F.Cu at (131.2, 38.6)
- added C6: 10u, Capacitor_SMD:C_0603_1608Metric_Pad1.08x0.95mm_HandSolder, F.Cu at (29.8, 141.2)
- added C7: 0.1u, Capacitor_SMD:C_0603_1608Metric_Pad1.08x0.95mm_HandSolder, F.Cu at (131.2, 41.1)
- added C8: 0.1u, Capacitor_SMD:C_0603_1608Metric_Pad1.08x0.95mm_HandSolder, F.Cu at (153.8, 36.0)
- added C9: 0.1u, Capacitor_SMD:C_0603_1608Metric_Pad1.08x0.95mm_HandSolder, F.Cu at (155.5, 21.8)
- added D1: LED, Diode_SMD:D_0805_2012Metric_Pad1.15x1.40mm_HandSolder, F.Cu at (62.2, 136.6)
- added D2: LED, Diode_SMD:D_0805_2012Metric_Pad1.15x1.40mm_HandSolder, F.Cu at (61.8, 131.2)
- added D3: LED, Diode_SMD:D_0805_2012Metric_Pad1.15x1.40mm_HandSolder, F.Cu at (62.0, 126.7)
- added Encoder1: Conn_01x04_Pin, Connector_JST:JST_XH_B4B-XH-A_1x04_P2.50mm_Vertical, F.Cu at (79.8, 109.8)
- added Encoder2: Conn_01x04_Pin, Connector_JST:JST_XH_B4B-XH-A_1x04_P2.50mm_Vertical, F.Cu at (79.3, 100.2)
- added Encoder3: Conn_01x04_Pin, Connector_JST:JST_XH_B4B-XH-A_1x04_P2.50mm_Vertical, F.Cu at (79.7, 90.0)
- added F1: Polyfuse, Fuse:Fuse_0603_1608Metric_Pad1.05x0.95mm_HandSolder, F.Cu at (77.5, 124.9)
- added F2: Polyfuse, Fuse:Fuse_0603_1608Metric_Pad1.05x0.95mm_HandSolder, F.Cu at (77.5, 127.4)
- added F3: Polyfuse, Fuse:Fuse_0603_1608Metric_Pad1.05x0.95mm_HandSolder, F.Cu at (77.5, 129.9)
- added H5: MountingHole_Pad, MountingHole:MountingHole_4.3mm_M4_DIN965_Pad_TopBottom, F.Cu at (119.6, 185.9)
- added H6: MountingHole_Pad, MountingHole:MountingHole_4.3mm_M4_DIN965_Pad_TopBottom, F.Cu at (132.3, 185.9)
- added H7: MountingHole_Pad, MountingHole:MountingHole_4.3mm_M4_DIN965_Pad_TopBottom, F.Cu at (145.0, 185.9)
- added H8: MountingHole_Pad, MountingHole:MountingHole_4.3mm_M4_DIN965_Pad_TopBottom, F.Cu at (156.4, 185.9)
- added IB2: ~, MyCustoms:Isobuck, F.Cu at (167.8, 102.2)
- added J10: MAIN KILL, Connector_AMASS:AMASS_XT30U-M_1x02_P5.0mm_Vertical, F.Cu at (220.8, 88.0)
- added J11: BatteryIN, Connector_AMASS:AMASS_XT30U-M_1x02_P5.0mm_Vertical, F.Cu at (234.4, 95.1)
- added J12: Conn_01x06_Pin, Connector_JST:JST_XH_B6B-XH-A_1x06_P2.50mm_Vertical, F.Cu at (75.7, 40.3)
- added J13: MOTOR 2 PWR, Connector_AMASS:AMASS_XT30U-M_1x02_P5.0mm_Vertical, F.Cu at (197.7, 74.7)
- added J14: MOTOR 4 PWR, Connector_AMASS:AMASS_XT30U-M_1x02_P5.0mm_Vertical, F.Cu at (189.2, 74.5)
- added J15: 24V TO 5V BUCK IN, Connector_AMASS:AMASS_XT30U-M_1x02_P5.0mm_Vertical, F.Cu at (206.2, 75.0)
- added J16: Conn_01x04_Pin, Connector_JST:JST_XH_B4B-XH-A_1x04_P2.50mm_Vertical, F.Cu at (89.8, 27.5)
- added J17: BASE KILL, Connector_AMASS:AMASS_XT30U-M_1x02_P5.0mm_Vertical, F.Cu at (207.2, 88.4)
- added J18: 24V TO 12V BUCK IN, Connector_AMASS:AMASS_XT30U-M_1x02_P5.0mm_Vertical, F.Cu at (214.3, 74.9)
- added J19: COOLING SYSTEM, Connector_AMASS:AMASS_XT30U-M_1x02_P5.0mm_Vertical, F.Cu at (188.8, 104.2)
- added J20: COOLING SYSTEM, Connector_AMASS:AMASS_XT30U-M_1x02_P5.0mm_Vertical, F.Cu at (179.0, 111.5)
- added J21: 24V TO 5V BUCK OUT, Connector_AMASS:AMASS_XT30U-M_1x02_P5.0mm_Vertical, F.Cu at (213.1, 111.1)
- added J22: 24V TO 12V BUCK OUT, Connector_AMASS:AMASS_XT30U-M_1x02_P5.0mm_Vertical, F.Cu at (197.6, 111.7)
- added J23: ARM KILL 24V, Connector_AMASS:AMASS_XT30U-M_1x02_P5.0mm_Vertical, F.Cu at (207.9, 95.8)
- added J24: JETSON KILL, Connector_AMASS:AMASS_XT30U-M_1x02_P5.0mm_Vertical, F.Cu at (226.1, 95.7)
- added J25: ARM KILL 12V, Connector_AMASS:AMASS_XT30U-M_1x02_P5.0mm_Vertical, F.Cu at (169.8, 96.2)
- added J26: BASE MOTOR KILL, Connector_AMASS:AMASS_XT30U-M_1x02_P5.0mm_Vertical, F.Cu at (194.0, 88.8)
- added J27: EXTRA 12V PORT, Connector_AMASS:AMASS_XT30U-M_1x02_P5.0mm_Vertical, F.Cu at (188.9, 96.1)
- added J28: EXTRA 5V PORT, Connector_AMASS:AMASS_XT30U-M_1x02_P5.0mm_Vertical, F.Cu at (213.1, 103.3)
- added J29: EXTRA 24V PORT, Connector_AMASS:AMASS_XT30U-M_1x02_P5.0mm_Vertical, F.Cu at (227.7, 79.8)
- added J3: Conn_01x01_Pin, Connector_PinHeader_2.54mm:PinHeader_1x01_P2.54mm_Vertical, F.Cu at (40.7, 44.0)
- added J30: Conn_01x02_Pin, Connector_JST:JST_XH_B2B-XH-A_1x02_P2.50mm_Vertical, F.Cu at (146.5, 98.2)
- added J31: Conn_01x02_Pin, Connector_JST:JST_XH_B2B-XH-A_1x02_P2.50mm_Vertical, F.Cu at (154.4, 98.2)
- added J32: Conn_01x02_Pin, Connector_JST:JST_XH_B2B-XH-A_1x02_P2.50mm_Vertical, F.Cu at (162.2, 98.2)
- added J34: Conn_01x03_Pin, Connector_JST:JST_XH_B3B-XH-A_1x03_P2.50mm_Vertical, F.Cu at (41.9, 63.5)
- added J35: Conn_01x03_Pin, Connector_JST:JST_XH_B3B-XH-A_1x03_P2.50mm_Vertical, F.Cu at (42.4, 82.1)
- added J36: Conn_01x03_Pin, Connector_JST:JST_XH_B3B-XH-A_1x03_P2.50mm_Vertical, F.Cu at (41.9, 73.1)
- added J4: Conn_01x04_Pin, Connector_JST:JST_XH_B4B-XH-A_1x04_P2.50mm_Vertical, F.Cu at (90.1, 49.6)
- added J5: Conn_01x06_Pin, Connector_JST:JST_XH_B6B-XH-A_1x06_P2.50mm_Vertical, F.Cu at (76.2, 60.4)
- added J6: MOTOR 1 PWR, Connector_AMASS:AMASS_XT30U-M_1x02_P5.0mm_Vertical, F.Cu at (179.5, 74.8)
- added J7: MOTOR 3 PWR, Connector_AMASS:AMASS_XT30U-M_1x02_P5.0mm_Vertical, F.Cu at (181.2, 88.2)
- added J8: STEPPER AND BLDC POWER, Connector_AMASS:AMASS_XT30U-M_1x02_P5.0mm_Vertical, F.Cu at (199.8, 102.2)
- added J9: JETSON POWER, Connector_AMASS:AMASS_XT30U-M_1x02_P5.0mm_Vertical, F.Cu at (222.5, 103.5)
- added MD1: Conn_01x03_Pin, Connector_JST:JST_XH_B3B-XH-A_1x03_P2.50mm_Vertical, F.Cu at (-18.0, 85.4)
- added MD2: Conn_01x03_Pin, Connector_JST:JST_XH_B3B-XH-A_1x03_P2.50mm_Vertical, F.Cu at (-18.1, 95.7)
- added MD3: Conn_01x03_Pin, Connector_JST:JST_XH_B3B-XH-A_1x03_P2.50mm_Vertical, F.Cu at (-17.9, 105.5)
- added MD4: Conn_01x03_Pin, Connector_JST:JST_XH_B3B-XH-A_1x03_P2.50mm_Vertical, F.Cu at (-17.9, 114.5)
- added R1: 1K, Resistor_SMD:R_0603_1608Metric_Pad0.98x0.95mm_HandSolder, F.Cu at (58.6, 136.7)
- added R2: 220, Resistor_SMD:R_0603_1608Metric_Pad0.98x0.95mm_HandSolder, F.Cu at (58.3, 131.2)
- added R3: 1K, Resistor_SMD:R_0603_1608Metric_Pad0.98x0.95mm_HandSolder, F.Cu at (58.4, 126.5)
- added R4: 2k2, Resistor_SMD:R_0603_1608Metric_Pad0.98x0.95mm_HandSolder, F.Cu at (169.0, 52.3)
- added R5: 2k2, Resistor_SMD:R_0603_1608Metric_Pad0.98x0.95mm_HandSolder, F.Cu at (166.4, 53.6)
- added R6: 2k2, Resistor_SMD:R_0603_1608Metric_Pad0.98x0.95mm_HandSolder, F.Cu at (152.7, 51.0)
- added R7: 2k2, Resistor_SMD:R_0603_1608Metric_Pad0.98x0.95mm_HandSolder, F.Cu at (153.4, 54.4)
- added R8: 10k, Resistor_SMD:R_0603_1608Metric_Pad0.98x0.95mm_HandSolder, F.Cu at (131.2, 43.6)
- added R9: 10k, Resistor_SMD:R_0603_1608Metric_Pad0.98x0.95mm_HandSolder, F.Cu at (131.2, 46.2)
- added STM1: STM32F411_BP, MyCustoms:blackpill_fp, F.Cu at (103.0, 117.9)
- added U1: ISO1540, Package_SO:SOIC-8_3.9x4.9mm_P1.27mm, F.Cu at (159.8, 52.7)
- added U2: ISO7721D, Package_SO:SOIC-8_3.9x4.9mm_P1.27mm, F.Cu at (152.4, 29.2)
- added U3: ISO7640FMDW, MyCustoms:ISO7640FMDW(SOIC127P1030X265-16N), F.Cu at (122.8, 42.2)
- added U4: AMS1117-3.3, Package_TO_SOT_SMD:SOT-223-3_TabPin2, F.Cu at (35.9, 140.4)
- moved J1 97.4 mm to (88.0, 93.5), turned to 0 degrees
- moved J2 73.6 mm to (116.3, 93.2), turned to 0 degrees
Connections:
- net GND1 renamed GND
- J1 pad 1: unconnected-(J1-Pin_1-Pad1) -> M4DIR
- J1 pad 10: STM1_TX -> ENC3A
- J1 pad 11: BNO_SDA -> ENC3B
- J1 pad 12: SYNC_CLK_OUT -> ENC2A
- J1 pad 13: unconnected-(J1-Pin_13-Pad13) -> ENC2B
- J1 pad 14: unconnected-(J1-Pin_14-Pad14) -> ENC1A
- J1 pad 15: unconnected-(J1-Pin_15-Pad15) -> ENC1B
- J1 pad 16: unconnected-(J1-Pin_16-Pad16) -> SDA_STM
- J1 pad 18: Net-(J1-Pin_18) -> unconnected-(J1-Pin_18-Pad18)
- J1 pad 20: unconnected-(J1-Pin_20-Pad20) -> +3.3V
- J1 pad 3: unconnected-(J1-Pin_3-Pad3) -> MISO_STM
- J1 pad 4: unconnected-(J1-Pin_4-Pad4) -> MOSI_STM
- J1 pad 5: unconnected-(J1-Pin_5-Pad5) -> SCL_STM
- J1 pad 6: unconnected-(J1-Pin_6-Pad6) -> CS2_STM
- J1 pad 7: STM1_RX -> CS1_STM
- J2 pad 1: Net-(J2-Pin_1) -> unconnected-(J2-Pin_1-Pad1)
- J2 pad 10: unconnected-(J2-Pin_10-Pad10) -> ISENSE_3
- J2 pad 12: unconnected-(J2-Pin_12-Pad12) -> M4PWM
- J2 pad 13: unconnected-(J2-Pin_13-Pad13) -> M3PWM
- J2 pad 14: unconnected-(J2-Pin_14-Pad14) -> M2PWM
- J2 pad 15: unconnected-(J2-Pin_15-Pad15) -> M1PWM
- J2 pad 19: unconnected-(J2-Pin_19-Pad19) -> LW_LED_STM
- J2 pad 3: 3.3V_STM_1 -> +3.3V
- J2 pad 4: BNO_SCL -> CLK_STM
- J2 pad 5: unconnected-(J2-Pin_5-Pad5) -> M3DIR
- J2 pad 6: unconnected-(J2-Pin_6-Pad6) -> M2DIR
- J2 pad 7: unconnected-(J2-Pin_7-Pad7) -> M1DIR
- J2 pad 8: unconnected-(J2-Pin_8-Pad8) -> ISENSE_1
- J2 pad 9: unconnected-(J2-Pin_9-Pad9) -> ISENSE_2

Commit message: Layout Components
Parts:
- removed H7: MountingHole_Pad, MountingHole:MountingHole_4.3mm_M4_DIN965_Pad_TopBottom
- removed J19, J20: COOLING SYSTEM, Connector_AMASS:AMASS_XT30U-M_1x02_P5.0mm_Vertical
- removed J3: Conn_01x01_Pin, Connector_PinHeader_2.54mm:PinHeader_1x01_P2.54mm_Vertical
- removed J31, J32: Conn_01x02_Pin, Connector_JST:JST_XH_B2B-XH-A_1x02_P2.50mm_Vertical
- removed J35, J36: Conn_01x03_Pin, Connector_JST:JST_XH_B3B-XH-A_1x03_P2.50mm_Vertical
- added R11: 6R8K, Resistor_SMD:R_0603_1608Metric_Pad0.98x0.95mm_HandSolder, B.Cu at (112.2, 73.3)
- added R12: 6R8K, Resistor_SMD:R_0603_1608Metric_Pad0.98x0.95mm_HandSolder, B.Cu at (110.8, 74.8)
- added R13: 6R8K, Resistor_SMD:R_0603_1608Metric_Pad0.98x0.95mm_HandSolder, B.Cu at (121.3, 74.3)
- added R14: 6R8K, Resistor_SMD:R_0603_1608Metric_Pad0.98x0.95mm_HandSolder, B.Cu at (125.0, 72.8)
- added R15: 6R8K, Resistor_SMD:R_0603_1608Metric_Pad0.98x0.95mm_HandSolder, B.Cu at (140.0, 73.4)
- added R16: 6R8K, Resistor_SMD:R_0603_1608Metric_Pad0.98x0.95mm_HandSolder, B.Cu at (137.6, 74.9)
- C1, C11, C13, C2, C5, C7, C8, C9, F1, F2, F3, R4, R5, R6, R7, R8, R9, U4: moved to B.Cu
- H5, H6: footprint MountingHole:MountingHole_4.3mm_M4_DIN965_Pad_TopBottom -> MountingHole:MountingHole_4.3mm_M4_ISO14580_Pad
- IB2: footprint MyCustoms:Isobuck -> Connector_PinHeader_2.54mm:PinHeader_1x04_P2.54mm_Vertical
- J10, J11: footprint Connector_AMASS:AMASS_XT30U-M_1x02_P5.0mm_Vertical -> Connector_AMASS:AMASS_XT60-M_1x02_P7.20mm_Vertical
- moved MD4 164.8 mm to (146.9, 110.7), turned to 180 degrees
- moved MD3 149.1 mm to (131.1, 110.8), turned to 180 degrees
- moved J22 146.6 mm to (65.4, 48.1), turned to 0 degrees
- moved H5 141.6 mm to (78.3, 50.5)
- moved MD2 136.3 mm to (117.3, 110.9), turned to 180 degrees
- moved H6 135.6 mm to (139.1, 50.5)
- moved D1 124.4 mm to (168.1, 71.3)
- moved D3 124.4 mm to (167.8, 61.3)
- moved R2 124.4 mm to (164.2, 65.9)
- moved D2 124.4 mm to (167.6, 65.8)
- moved R1 124.4 mm to (164.4, 71.4)
- moved R3 124.4 mm to (164.2, 61.2)
- moved MD1 123.3 mm to (102.7, 110.9), turned to 180 degrees
- moved J6 119.8 mm to (64.8, 40.1), turned to 0 degrees
- moved H8 114.9 mm to (78.3, 101.7)
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Connections:
- net ISENSE_2 renamed Net-(J2-Pin_9)
- B2 pad 11: Net-(B2-INT) -> unconnected-(B2-INT-Pad11)
- B2 pad 16: unconnected-(B2-3V3-Pad16) -> 3.3V_ISO_BNO
- B2 pad 2: 3.3V_ISO_BNO -> unconnected-(B2-3V3-Pad2)
- J1 pad 1: M4DIR -> ISENSE
- J2 pad 10: ISENSE_3 -> unconnected-(J2-Pin_10-Pad10)
- J2 pad 5: M3DIR -> M4DIR
- J2 pad 6: M2DIR -> M3DIR
- J2 pad 7: M1DIR -> M2DIR
- J2 pad 8: ISENSE_1 -> M1DIR
- J34 pad 1: ISENSE_1 -> ISENSE
- STM1 pad 10: ISENSE_3 -> unconnected-(J2-Pin_10-Pad10)
- STM1 pad 21: M4DIR -> ISENSE
- STM1 pad 5: M3DIR -> M4DIR
- STM1 pad 6: M2DIR -> M3DIR
- STM1 pad 7: M1DIR -> M2DIR
- STM1 pad 8: ISENSE_1 -> M1DIR
