File: base_pcb.kicad_sch (KiCad schematic)
At the start: 41 parts, among them J1 Conn_01x20_Pin, J12 Conn_01x06_Pin, J16 Conn_01x04_Pin, J2 Conn_01x20_Pin, J3 Conn_01x01_Pin, J4 Conn_01x04_Pin, J5 Conn_01x06_Pin, U1 ISO1540, U2 ISO7721D, U3 ISO7640FMDW, U4 AMS1117-3.3

Commit message: Final Schematic
Parts:
- removed C3, C4: 0.1u, symbol Device:C_Small
- added C11, C13: 0.1u, Capacitor_SMD:C_0603_1608Metric_Pad1.08x0.95mm_HandSolder, symbol Device:C_Small
- added J34, J35, J36: Conn_01x03_Pin, symbol Connector:Conn_01x03_Pin
- added R8, R9: 10k, symbol Device:R_Small_US
- B2: footprint (none) -> MyCustoms:BNO085
- C2, C5, C7, C8, C9: footprint (none) -> Capacitor_SMD:C_0603_1608Metric_Pad1.08x0.95mm_HandSolder
- renumbered MotorController1 to STM1
Connections:
- net +3.3V: now also C11.2, R8.2, R9.1
- net +5V: now also J34.2 (Pin_2), J35.2 (Pin_2), J36.2 (Pin_2)
- net 3.3V_ISO: now also C13.2
- net CLK_STM: now also J2.4 (Pin_4), STM1.4 (PB10)
- net CS1_STM: now also J1.7 (Pin_7), STM1.27 (PA10), R9.2
- net CS2_STM: now also J1.6 (Pin_6), STM1.26 (PA9), R8.1
- net GND: now also C11.1, J34.3 (Pin_3), J35.3 (Pin_3), J36.3 (Pin_3)
- net ISOGND: now also C13.1
- net LW_LED_STM: now also J2.19 (Pin_19), STM1.19 (PC13)
- net MISO_STM: now also J1.3 (Pin_3), STM1.23 (PB14)
- net MOSI_STM: now also J1.4 (Pin_4), STM1.24 (PB15)
- net SCL_STM: now also J1.5 (Pin_5), STM1.25 (PA8)
- net SDA_STM: now also J1.16 (Pin_16), STM1.36 (PB8)
- net ISENSE_3: now reaches J2.10 (Pin_10), STM1.10 (PA5)
- net ISENSE_3: now also J36.1 (Pin_1)
- net ISENSE_2: now reaches J2.9 (Pin_9), STM1.9 (PA6)
- net ISENSE_2: now also J35.1 (Pin_1)
- net ISENSE renamed ISENSE_1
- net ISENSE_1: now also J34.1 (Pin_1)
Other:
- note added: "CONTROLLER"
- note added: "Current Sensors"
- note added: "Decoupling Capacitors"
- note added: "ISOLATORS"
- note added: "MOTOR"
- note added: "POWER"
- note added: "SENSORS"
- moved on the sheet: B2, C1, C10, C2, C5, C6, C7, C8, D1, D2, D3, Encoder1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

Commit message: Add STM pinouts
Parts:
- added F1, F2, F3: Polyfuse, Fuse:Fuse_0603_1608Metric_Pad1.05x0.95mm_HandSolder, symbol Device:Polyfuse
- C1: footprint (none) -> Capacitor_SMD:C_0603_1608Metric_Pad1.08x0.95mm_HandSolder
- IB2: footprint (none) -> Connector_PinHeader_2.54mm:PinHeader_1x04_P2.54mm_Vertical
- J12, J5: footprint (none) -> Connector_JST:JST_XH_B6B-XH-A_1x06_P2.50mm_Vertical
- J16, J4: footprint (none) -> Connector_JST:JST_XH_B4B-XH-A_1x04_P2.50mm_Vertical
- J3: footprint (none) -> Connector_PinHeader_2.54mm:PinHeader_1x01_P2.54mm_Vertical
- J34, J35, J36: footprint (none) -> Connector_JST:JST_XH_B3B-XH-A_1x03_P2.50mm_Vertical
- R1, R2, R3: footprint PCM_Resistor_SMD_AKL:R_0603_1608Metric_Pad0.98x0.95mm_HandSolder -> Resistor_SMD:R_0603_1608Metric_Pad0.98x0.95mm_HandSolder
- R4, R5, R6, R7, R8, R9: footprint (none) -> Resistor_SMD:R_0603_1608Metric_Pad0.98x0.95mm_HandSolder
- STM1: footprint ROBO:STM32F411-BP -> MyCustoms:blackpill_fp
- U3: footprint ISO7640FMDW:SOIC127P1030X265-16N -> MyCustoms:ISO7640FMDW(SOIC127P1030X265-16N)
- renumbered MDD1 to MD1, MDD2 to MD2, MDD3 to MD3, MDD4 to MD4
Connections:
- net 3.3V_ISO: now also F1.1, F2.1, F3.1; no longer B2.2 (3V3), J12.4 (Pin_4), J5.4 (Pin_4)
- net CLK: now also U3.13 (OUTB); no longer U3.4 (INB)
- net CLK_STM: now also U3.4 (INB); no longer U3.13 (OUTB)
- net CS1: now also U3.14 (OUTA); no longer U3.3 (INA)
- net CS1_STM: now also U3.3 (INA); no longer U3.14 (OUTA)
- net CS2: now also U3.11 (OUTD); no longer U3.6 (IND)
- net CS2_STM: now also U3.6 (IND); no longer U3.11 (OUTD)
- net LW_LED: now also U3.12 (OUTC); no longer U3.5 (INC)
- net LW_LED_STM: now also U3.5 (INC); no longer U3.12 (OUTC)
- new net 3.3V_ISO_BNO: B2.2 (3V3), F1.2
- new net 3.3V_ISO_LW1: F2.2, J5.4 (Pin_4)
- new net 3.3V_ISO_LW2: F3.2, J12.4 (Pin_4)
- no-connect marks 13 -> 20
Other:
- note added: "Fuses"
- note added: "LiteWing Modules"
- note added: "PORTS"
- note removed: "LiteWing Module"
- moved on the sheet: B2, C1, C10, C2, C5, C6, C7, D1, D2, D3, IB2, J12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

Commit message: Layout Components
Parts:
- removed J3: Conn_01x01_Pin, Connector_PinHeader_2.54mm:PinHeader_1x01_P2.54mm_Vertical, symbol Connector:Conn_01x01_Pin
- removed J35, J36: Conn_01x03_Pin, Connector_JST:JST_XH_B3B-XH-A_1x03_P2.50mm_Vertical, symbol Connector:Conn_01x03_Pin
- added R11, R12, R13, R14, R15, R16: 6R8K, Resistor_SMD:R_0603_1608Metric_Pad0.98x0.95mm_HandSolder, symbol Device:R_Small_US
Connections:
- net 3.3V_ISO_BNO: now also B2.16 (3V3); no longer B2.2 (3V3)
- net 5V: now also R11.2, R12.2, R13.2, R14.2, R15.2, R16.2
- net ENC1A: now also R11.1
- net ENC1B: now also R12.1
- net ENC2A: now also R14.1
- net ENC2B: now also R13.1
- net ENC3A: now also R15.1
- net ENC3B: now also R16.1
- net M1DIR: now also J2.8 (Pin_8), STM1.8 (PA7); no longer J2.7 (Pin_7), STM1.7 (PB0)
- net M2DIR: now also J2.7 (Pin_7), STM1.7 (PB0); no longer J2.6 (Pin_6), STM1.6 (PB1)
- net M3DIR: now also J2.6 (Pin_6), STM1.6 (PB1); no longer J2.5 (Pin_5), STM1.5 (PB2)
- net M4DIR: now also J2.5 (Pin_5), STM1.5 (PB2); no longer J1.1 (Pin_1), STM1.21 (PB12)
- removed net ISENSE_1: J2.8 (Pin_8), J34.1 (Pin_1), STM1.8 (PA7)
- net ISENSE_2: no longer names the net of J2.9 (Pin_9), STM1.9 (PA6)
- net ISENSE_3: no longer names the net of J2.10 (Pin_10), STM1.10 (PA5)
- new net ISENSE: J1.1 (Pin_1), J34.1 (Pin_1), STM1.21 (PB12)
- no-connect marks 20 -> 22
Other:
- note added: "Current Sensor"
- note added: "Encoder Pull Up"
- note removed: "Current Sensors"
- moved on the sheet: B2, Encoder1, Encoder2, Encoder3, J34, MD1, MD2, MD3, MD4
