File: ports.kicad_sch (KiCad schematic)
At the start: 30 parts, among them J10 MAIN KILL, J11 BatteryIN, J13 MOTOR 2 PWR, J14 MOTOR 4 PWR, J15 24V TO 5V BUCK IN, J17 BASE KILL, J18 24V TO 12V BUCK IN, J19 COOLING SYSTEM, J20 COOLING SYSTEM, J21 24V TO 5V BUCK OUT, J22 24V TO 12V BUCK OUT, J23 ARM KILL 24V, J24 JETSON KILL, J25 ARM KILL 24V, J26 BASE KILL, J27 EXTRA 12V PORT, J28 EXTRA 5V PORT, J29 EXTRA 24V PORT, J30 EXTRA 3.3V PORT, J31 Conn_01x03_Pin, J32 Conn_01x03_Pin, J33 Conn_01x03_Pin, J6 MOTOR 1 PWR, J7 MOTOR 3 PWR, J8 STEPPER AND BLDC POWER, J9 JETSON POWER

Commit message: Add STM pinouts
Parts:
- removed J30: EXTRA 3.3V PORT, ROBO:xt60, symbol XT60-M:XT60-M
- removed J31, J32, J33: Conn_01x03_Pin, Connector_JST:JST_XH_B3B-XH-A_1x03_P2.50mm_Vertical, symbol Connector:Conn_01x03_Pin
- added J30, J31, J32: Conn_01x02_Pin, Connector_JST:JST_XH_B2B-XH-A_1x02_P2.50mm_Vertical, symbol Connector:Conn_01x02_Pin
- J10, J11, J13, J14, J15, J17, J18, J19, J20, J21, J22, J23, J24, J27, J28, J29, J6, J7, J8, J9: footprint ROBO:xt60 -> Connector_AMASS:AMASS_XT30U-M_1x02_P5.0mm_Vertical; symbol XT60-M:XT60-M -> customs:XT_connect
- J25: value ARM KILL 24V -> ARM KILL 12V; footprint ROBO:xt60 -> Connector_AMASS:AMASS_XT30U-M_1x02_P5.0mm_Vertical; symbol XT60-M:XT60-M -> customs:XT_connect
- J26: value BASE KILL -> BASE MOTOR KILL; footprint ROBO:xt60 -> Connector_AMASS:AMASS_XT30U-M_1x02_P5.0mm_Vertical; symbol XT60-M:XT60-M -> customs:XT_connect
Connections:
- net +12V: now also J19.2 (POS), J20.2 (POS), J22.2 (POS), J25.2 (POS), J27.2 (POS); no longer J19.P (POS), J20.P (POS), J22.P (POS), J25.P (POS), J27.P (POS)
- net +24V: now also J10.1 (NEG), J17.2 (POS), J18.2 (POS), J23.2 (POS), J24.2 (POS), J29.2 (POS); no longer J10.N (NEG), J17.P (POS), J18.P (POS), J23.P (POS), J24.P (POS), J29.P (POS)
- net +5V: now also J21.2 (POS), J28.2 (POS); no longer J21.P (POS), J28.P (POS)
- net 12V_ARM: now also J25.1 (NEG), J30.2 (Pin_2), J31.2 (Pin_2), J32.2 (Pin_2); no longer J25.N (NEG)
- net 24V_ARM: now also J23.1 (NEG), J8.2 (POS); no longer J23.N (NEG), J8.P (POS)
- net 24V_BASE: now also J15.2 (POS), J17.1 (NEG), J26.2 (POS); no longer J15.P (POS), J17.N (NEG), J26.P (POS)
- net 24V_BASE_M: now also J13.2 (POS), J14.2 (POS), J26.1 (NEG), J6.2 (POS), J7.2 (POS); no longer J13.P (POS), J14.P (POS), J6.P (POS), J7.P (POS)
- net 24V_BATTERY: now also J10.2 (POS), J11.2 (POS); no longer J10.P (POS), J11.P (POS)
- net 24V_Jetson: now also J24.1 (NEG), J9.2 (POS); no longer J24.N (NEG), J9.P (POS)
- net GND: now also J11.1 (NEG), J13.1 (NEG), J14.1 (NEG), J15.1 (NEG), J18.1 (NEG), J19.1 (NEG), J20.1 (NEG), J21.1 (NEG), J22.1 (NEG), J27.1 (NEG), J28.1 (NEG), J29.1 (NEG), J6.1 (NEG), J7.1 (NEG), J8.1 (NEG), J9.1 (NEG), J30.1 (Pin_1), J31.1 (Pin_1), J32.1 (Pin_1); no longer J11.N (NEG), J13.N (NEG), J14.N (NEG), J15.N (NEG), J18.N (NEG), J19.N (NEG), J20.N (NEG), J21.N (NEG), J22.N (NEG), J27.N (NEG), J28.N (NEG), J29.N (NEG), J6.N (NEG), J7.N (NEG), J8.N (NEG), J9.N (NEG)
- removed net 24V_BASE_Motors: J26.N (NEG)
Other:
- note added: "Stepper and BLDC Power"
- moved on the sheet: H5, H6, H7, H8

Commit message: Layout Components
Parts:
- removed H7: MountingHole_Pad, MountingHole:MountingHole_4.3mm_M4_DIN965_Pad_TopBottom, symbol Mechanical:MountingHole_Pad
- removed J19, J20: COOLING SYSTEM, Connector_AMASS:AMASS_XT30U-M_1x02_P5.0mm_Vertical, symbol customs:XT_connect
- removed J31, J32: Conn_01x02_Pin, Connector_JST:JST_XH_B2B-XH-A_1x02_P2.50mm_Vertical, symbol Connector:Conn_01x02_Pin
- H5, H6: footprint MountingHole:MountingHole_4.3mm_M4_DIN965_Pad_TopBottom -> MountingHole:MountingHole_4.3mm_M4_ISO14580_Pad
- J10, J11: footprint Connector_AMASS:AMASS_XT30U-M_1x02_P5.0mm_Vertical -> Connector_AMASS:AMASS_XT60-M_1x02_P7.20mm_Vertical
Other:
- note added: "ARM PCB Power"
- note removed: "COOLING FANS"
- moved on the sheet: H5, H6, H8, J11, J27, J28, J29, J30, J9
